File: sparkfun_drone/sparkfun_drone.kicad_sch (KiCad schematic)
At the start: 5 parts

Commit message: new branch with fixes
Parts:
- removed J1: ~, SparkFun-MicroMod:M.2-CARD-E-22, symbol SparkFun-MicroMod:MICROMOD-2222
- removed M1, M2, M3, M4: ~, Library:1104_motor, symbol Motor:1104_motor
Other:
- added sheet Micromod (micromod.kicad_sch)
- added sheet Motors (motors.kicad_sch)
